Commit message: robot.urdf.xacro

File: src/mecanum_drive/urdf/robot.urdf.xacro (robot description, xacro)
@@ -1,20 +1,131 @@
+<?xml version="1.0"?>
 <robot xmlns:xacro="http://ros.org/wiki/xacro" name="mecanum_bot">
+  <!-- Use simulation time -->
+  <xacro:arg name="use_sim_time" default="true"/>
+  <!-- Parameters -->
   <xacro:property name="wheel_radius" value="0.05"/>
   <xacro:property name="wheel_separation_x" value="0.5"/>
   <xacro:property name="wheel_separation_y" value="0.5"/>
+  <!-- Base link -->
   <link name="base_link">
-    <visual><geometry><box size="0.6 0.6 0.1"/></geometry></visual>
+    <visual>
+      <geometry>
+        <box size="0.6 0.6 0.1"/>
+      </geometry>
+      <material name="gray">
+        <color rgba="0.5 0.5 0.5 1"/>
+      </material>
+    </visual>
+    <collision>
+      <geometry>
+        <box size="0.6 0.6 0.1"/>
+      </geometry>
+    </collision>
+    <inertial>
+      <mass value="10.0"/>
+      <inertia ixx="1.0" ixy="0.0" ixz="0.0" iyy="1.0" iyz="0.0" izz="1.0"/>
+    </inertial>
   </link>
+  <!-- Wheel Macro -->
+  <xacro:macro name="mecanum_wheel" params="prefix x y joint_name">
+    <link name="${prefix}_wheel">
+      <visual>
+        <geometry>
+          <cylinder radius="${wheel_radius}" length="0.05"/>
+        </geometry>
+        <material name="black">
+          <color rgba="0.1 0.1 0.1 1"/>
+        </material>
+      </visual>
+      <collision>
+        <geometry>
+          <cylinder radius="${wheel_radius}" length="0.05"/>
+        </geometry>
+      </collision>
+      <inertial>
+        <mass value="1.0"/>
+        <inertia ixx="0.1" ixy="0.0" ixz="0.0" iyy="0.1" iyz="0.0" izz="0.1"/>
+      </inertial>
+    </link>
+    <joint name="${joint_name}" type="continuous">
+      <parent link="base_link"/>
+      <child link="${prefix}_wheel"/>
+      <origin xyz="${x} ${y} 0" rpy="0 1.5707 0"/>
+      <axis xyz="0 0 1"/>
+      <limit effort="1.0" velocity="100.0"/>
+      <dynamics damping="0.0" friction="0.0"/>
+    </joint>
+  </xacro:macro>
+  <!-- Wheels -->
+  <xacro:mecanum_wheel prefix="front_left"  x="${-wheel_separation_x/2}" y="${wheel_separation_y/2}"  joint_name="front_left_joint"/>
+  <xacro:mecanum_wheel prefix="front_right" x="${wheel_separation_x/2}"  y="${wheel_separation_y/2}"  joint_name="front_right_joint"/>
+  <xacro:mecanum_wheel prefix="rear_left"   x="${-wheel_separation_x/2}" y="${-wheel_separation_y/2}" joint_name="rear_left_joint"/>
+  <xacro:mecanum_wheel prefix="rear_right"  x="${wheel_separation_x/2}"  y="${-wheel_separation_y/2}" joint_name="rear_right_joint"/>
+  <!-- Gazebo plugin for ros2_control -->
   <gazebo>
-    <plugin name="diff_drive_controller" filename="libgazebo_ros_diff_drive.so">
-      <ros>
-        <remapping>cmd_vel:=/cmd_vel</remapping>
-      </ros>
-      <update_rate>100</update_rate>
-      <wheel_separation>${wheel_separation_x}</wheel_separation>
-      <wheel_diameter>${2 * wheel_radius}</wheel_diameter>
-      <left_joint>left_wheel_joint</left_joint>
-      <right_joint>right_wheel_joint</right_joint>
-    </plugin>
+    <plugin name="gazebo_ros2_control" filename="libgazebo_ros2_control.so"/>
   </gazebo>
+  <!-- ros2_control configuration -->
+  <ros2_control name="MecanumHardware" type="system">
+    <hardware>
+      <plugin>gazebo_ros2_control/GazeboSystem</plugin>
+    </hardware>
+    <joint name="front_left_joint">
+      <command_interface name="velocity"/>
+      <state_interface name="position"/>
+      <state_interface name="velocity"/>
+    </joint>
+    <joint name="front_right_joint">
+      <command_interface name="velocity"/>
+      <state_interface name="position"/>
+      <state_interface name="velocity"/>
+    </joint>
+    <joint name="rear_left_joint">
+      <command_interface name="velocity"/>
+      <state_interface name="position"/>
+      <state_interface name="velocity"/>
+    </joint>
+    <joint name="rear_right_joint">
+      <command_interface name="velocity"/>
+      <state_interface name="position"/>
+      <state_interface name="velocity"/>
+    </joint>
+  </ros2_control>
+  <!-- Transmissions -->
+  <transmission name="front_left_trans">
+    <type>transmission_interface/SimpleTransmission</type>
+    <joint name="front_left_joint">
+      <hardwareInterface>hardware_interface/VelocityJointInterface</hardwareInterface>
+    </joint>
+    <actuator name="motor_front_left">
+      <mechanicalReduction>1</mechanicalReduction>
+    </actuator>
+  </transmission>
+  <transmission name="front_right_trans">
+    <type>transmission_interface/SimpleTransmission</type>
+    <joint name="front_right_joint">
+      <hardwareInterface>hardware_interface/VelocityJointInterface</hardwareInterface>
+    </joint>
+    <actuator name="motor_front_right">
+      <mechanicalReduction>1</mechanicalReduction>
+    </actuator>
+  </transmission>
+  <transmission name="rear_left_trans">
+    <type>transmission_interface/SimpleTransmission</type>
+    <joint name="rear_left_joint">
+      <hardwareInterface>hardware_interface/VelocityJointInterface</hardwareInterface>
+    </joint>
+    <actuator name="motor_rear_left">
+      <mechanicalReduction>1</mechanicalReduction>
+    </actuator>
+  </transmission>
+  <transmission name="rear_right_trans">
+    <type>transmission_interface/SimpleTransmission</type>
+    <joint name="rear_right_joint">
+      <hardwareInterface>hardware_interface/VelocityJointInterface</hardwareInterface>
+    </joint>
+    <actuator name="motor_rear_right">
+      <mechanicalReduction>1</mechanicalReduction>
+    </actuator>
+  </transmission>
 </robot>
